File: PCB/Modular System/ZTO-80 CPU/ZTO-80 CPU.kicad_pcb (KiCad board)
At the start: 2 copper layers, 99.1 x 57.1 mm, 27 parts, among them J1 ZTO-80 Bus, J2 Conn_01x02, J3 Conn_01x09, SW1 SW_Push, U1 Z80CPU, U2 74HCT04, U3 74HCT541, U4 74HCT541, U5 74HCT245, X1 CXO_DIP8

Commit message: Edited power LED resistor value
Parts:
- R1: value 200 -> 220

Commit message: Update ZTO-80 CPU.kicad_pcb
Routing:
- net GND: track 10.5 -> 8.89 mm

Commit message: Updates to PDFs and the SBC
Other:
- board text added: "ZTO-80 CPU"
- board text added: "v1.1"
- board text removed: "ZTO-80 CPU V1.1"
Changed lines of the file:
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@@
-(kicad_pcb (version 20171130) (host pcbnew "(5.1.6)-1")
+(kicad_pcb (version 20171130) (host pcbnew "(5.1.5)-3")
   (general
     (thickness 1.6)
@@
   (title_block
     (title "ZTO-80 CPU")
-    (date 2020-07-13)
+    (date 2020-08-11)
     (rev 1.1)
     (company "Jacob Hahn")
@@
     (38 B.Mask user)
     (39 F.Mask user)
-    (40 Dwgs.User user)
+    (40 Dwgs.User user hide)
     (41 Cmts.User user hide)
     (42 Eco1.User user)
@@
     )
   )
+  (gr_text v1.1 (at 172.085 115.57) (layer F.SilkS)
+    (effects (font (size 1.524 1.524) (thickness 0.2032)) (justify left))
+  )
   (gr_text VCC (at 189.865 66.675) (layer F.SilkS)
     (effects (font (size 1.016 1.016) (thickness 0.1524)) (justify right))
@@
     (effects (font (size 1.27 1.27) (thickness 0.15)))
   )
-  (gr_text BACK (at 193.04 91.44 90) (layer B.SilkS)
-    (effects (font (size 2.032 2.032) (thickness 0.2032)) (justify mirror))
-  )
   (gr_text JLCJLCJLCJLC (at 189.865 118.745) (layer B.SilkS)
     (effects (font (size 0.899998 0.899998) (thickness 0.159995)) (justify mirror))
@@
     (effects (font (size 1.524 1.524) (thickness 0.2032)))
   )
-  (gr_text "ZTO-80 CPU V1.1" (at 145.415 109.22) (layer F.SilkS)
+  (gr_text "ZTO-80 CPU" (at 145.415 109.855) (layer F.SilkS)
     (effects (font (size 2.54 2.54) (thickness 0.254)))
   )

Commit message: Changed bus orientation
This change is backwards-compatible with all previous ZTO-80 modules
Parts:
- J1: footprint ZTO-80_Header:PinHeader_2x20_P2.54mm_Horizontal -> Connector_PinHeader_2.54mm:PinHeader_2x20_P2.54mm_Horizontal
- moved J1 48.3 mm to (169.5, 113.7), turned to 270 degrees
Connections:
- J1 pad 1: /A15 -> /USR4
- J1 pad 10: /A6 -> /MREQ
- J1 pad 11: /A5 -> /INT
- J1 pad 12: /A4 -> /RST
- J1 pad 13: /A3 -> /M1
- J1 pad 14: /A2 -> /CLK
- J1 pad 15: /A1 -> /D0
- J1 pad 16: /A0 -> /D1
- J1 pad 17: VCC -> /D2
- J1 pad 18: GND -> /D3
- J1 pad 19: /D7 -> /D4
- J1 pad 2: /A14 -> /USR3
- J1 pad 20: /D6 -> /D5
- J1 pad 21: /D5 -> /D6
- J1 pad 22: /D4 -> /D7
- J1 pad 23: /D3 -> GND
- J1 pad 24: /D2 -> VCC
- J1 pad 25: /D1 -> /A0
- J1 pad 26: /D0 -> /A1
- J1 pad 27: /CLK -> /A2
- J1 pad 28: /M1 -> /A3
- J1 pad 29: /RST -> /A4
- J1 pad 3: /A13 -> /USR2
- J1 pad 30: /INT -> /A5
- J1 pad 31: /MREQ -> /A6
- J1 pad 32: /WR -> /A7
- J1 pad 33: /IORQ -> /A8
- J1 pad 34: /RD -> /A9
- J1 pad 35: /TXB -> /A10
- J1 pad 36: /RXB -> /A11
- J1 pad 37: /USR1 -> /A12
- J1 pad 38: /USR2 -> /A13
- J1 pad 39: /USR3 -> /A14
- J1 pad 4: /A12 -> /USR1
- J1 pad 40: /USR4 -> /A15
- J1 pad 5: /A11 -> /RXB
- J1 pad 6: /A10 -> /TXB
- J1 pad 7: /A9 -> /RD
- J1 pad 8: /A8 -> /IORQ
- J1 pad 9: /A7 -> /WR

Commit message: Added CERN license text to silkscreen
Other:
- board text added: "Licensed under CERN-OHL-S v2"
Changed lines of the file:
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@@
   (general
     (thickness 1.6)
-    (drawings 27)
+    (drawings 28)
     (tracks 487)
     (zones 0)
@@
     )
   )
+  (gr_text "Licensed under CERN-OHL-S v2" (at 109.22 118.745) (layer B.SilkS)
+    (effects (font (size 1 1) (thickness 0.15)) (justify mirror))
+  )
   (gr_text v1.1 (at 172.085 115.57) (layer F.SilkS)
