File: PCB/Modular System/ZTO-80 SIO/ZTO-80 SIO.kicad_pcb (KiCad board)
At the start: 2 copper layers, 99.1 x 57.1 mm, 34 parts, among them J1 ZTO-80 Bus, J2 Conn_01x02, J3 SIOHDR, J4 SIOHDR, SW1 SW_DIP_x06, U1 Z80SIO0, U2 74HC688, X1 1.8432MHz

Commit message: Added CERN license text to silkscreen
Other:
- board text added: "Licensed under CERN-OHL-S v2"
Changed lines of the file:
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@@
   (general
     (thickness 1.6)
-    (drawings 73)
+    (drawings 74)
     (tracks 364)
     (zones 0)
@@
     )
   )
+  (gr_text "Licensed under CERN-OHL-S v2" (at 108.712 118.872) (layer B.SilkS)
+    (effects (font (size 1 1) (thickness 0.15)) (justify mirror))
+  )
   (gr_text "BAUD CLOCK" (at 155.575 80.01) (layer F.SilkS)
     (effects (font (size 1 1) (thickness 0.15)))
@@
   (segment (start 142.875 101.6) (end 153.67 90.805) (width 0.254) (layer F.Cu) (net 7))
   (segment (start 153.67 90.805) (end 183.515 90.805) (width 0.254) (layer F.Cu) (net 7))
+  (via (at 170.18 90.805) (size 0.6096) (drill 0.3048) (layers F.Cu B.Cu) (net 7))
+  (segment (start 167.055801 93.929199) (end 170.18 90.805) (width 0.254) (layer B.Cu) (net 7))
+  (segment (start 167.055801 102.027081) (end 167.055801 93.929199) (width 0.254) (layer B.Cu) (net 7))
+  (segment (start 163.233999 108.546001) (end 163.233999 104.736001) (width 0.254) (layer B.Cu) (net 7))
+  (segment (start 161.925 109.855) (end 163.233999 108.546001) (width 0.254) (layer B.Cu) (net 7))
+  (segment (start 163.233999 104.736001) (end 165.188999 102.781001) (width 0.254) (layer B.Cu) (net 7))
+  (segment (start 165.188999 102.781001) (end 166.301881 102.781001) (width 0.254) (layer B.Cu) (net 7))
+  (segment (start 166.301881 102.781001) (end 167.055801 102.027081) (width 0.254) (layer B.Cu) (net 7))
   (segment (start 185.725 94.615) (end 186.3 94.615) (width 0.254) (layer F.Cu) (net 8))
   (segment (start 144.233999 101.988883) (end 144.233999 101.033119) (width 0.254) (layer F.Cu) (net 8))
@@
   (segment (start 145.453999 114.896001) (end 145.453999 110.928883) (width 0.254) (layer B.Cu) (net 24))
   (segment (start 144.145 116.205) (end 145.453999 114.896001) (width 0.254) (layer B.Cu) (net 24))
-  (via (at 170.18 90.805) (size 0.6096) (drill 0.3048) (layers F.Cu B.Cu) (net 7))
-  (segment (start 167.055801 93.929199) (end 170.18 90.805) (width 0.254) (layer B.Cu) (net 7))
-  (segment (start 167.055801 102.027081) (end 167.055801 93.929199) (width 0.254) (layer B.Cu) (net 7))
-  (segment (start 163.233999 108.546001) (end 163.233999 104.736001) (width 0.254) (layer B.Cu) (net 7))
-  (segment (start 161.925 109.855) (end 163.233999 108.546001) (width 0.254) (layer B.Cu) (net 7))
-  (segment (start 163.233999 104.736001) (end 165.188999 102.781001) (width 0.254) (layer B.Cu) (net 7))
-  (segment (start 165.188999 102.781001) (end 166.301881 102.781001) (width 0.254) (layer B.Cu) (net 7))
-  (segment (start 166.301881 102.781001) (end 167.055801 102.027081) (width 0.254) (layer B.Cu) (net 7))
   (segment (start 155.008119 100.418999) (end 156.933999 100.418999) (width 0.254) (layer F.Cu) (net 26))
   (segment (start 154.393999 101.033119) (end 155.008119 100.418999) (width 0.254) (layer F.Cu) (net 26))

Commit message: Finished SIO
Parts:
- R2, R3: value 100k -> 10k
Other:
- board text added: "2"
- board text added: "3"
- board text added: "4"
- board text added: "5"
- board text added: "6"
- board text added: "7"
- board text added: "Base Addresses: A Data: xxxxxx00 B Data: xxxxxx01 A Command: xxxxxx10 B Command: xxxxxx11"
