File: PCB/Modular System/ZTO-80 Backplane 5/ZTO-80 Backplane 5.kicad_pcb (KiCad board)
At the start: 2 copper layers, 99.1 x 91.4 mm, 33 parts, among them J1 ZTO-80 Bus, J10 Conn_01x02, J11 PJ-102A, J12 Conn_01x02, J13 Conn_01x02, J2 Conn_01x02, J3 ZTO-80 Bus, J4 Conn_01x02, J5 ZTO-80 Bus, J6 Conn_01x02, J7 ZTO-80 Bus, J8 Conn_01x02, J9 ZTO-80 Bus, SW1 Reset

Commit message: Edited power LED resistor value
Parts:
- R1: value 200 -> 220

Commit message: Changed bus orientation
This change is backwards-compatible with all previous ZTO-80 modules
Parts:
- moved J1 48.3 mm to (167.6, 62.2), turned to 270 degrees
- moved J3 48.3 mm to (167.6, 77.5), turned to 270 degrees
- moved J5 48.3 mm to (167.6, 92.7), turned to 270 degrees
- moved J7 48.3 mm to (167.6, 108.0), turned to 270 degrees
- moved J9 48.3 mm to (167.6, 123.2), turned to 270 degrees
Connections:
- J1 pad 1: /A15 -> /USR4
- J1 pad 10: /A6 -> /MREQ
- J1 pad 11: /A5 -> /INT
- J1 pad 12: /A4 -> /RST
- J1 pad 13: /A3 -> /M1
- J1 pad 14: /A2 -> /CLK
- J1 pad 15: /A1 -> /D0
- J1 pad 16: /A0 -> /D1
- J1 pad 17: VCC -> /D2
- J1 pad 18: GND -> /D3
- J1 pad 19: /D7 -> /D4
- J1 pad 2: /A14 -> /USR3
- J1 pad 20: /D6 -> /D5
- J1 pad 21: /D5 -> /D6
- J1 pad 22: /D4 -> /D7
- J1 pad 23: /D3 -> GND
- J1 pad 24: /D2 -> VCC
- J1 pad 25: /D1 -> /A0
- J1 pad 26: /D0 -> /A1
- J1 pad 27: /CLK -> /A2
- J1 pad 28: /M1 -> /A3
- J1 pad 29: /RST -> /A4
- J1 pad 3: /A13 -> /USR2
- J1 pad 30: /INT -> /A5
- J1 pad 31: /MREQ -> /A6
- J1 pad 32: /WR -> /A7
- J1 pad 33: /IORQ -> /A8
- J1 pad 34: /RD -> /A9
- J1 pad 35: /TXB -> /A10
- J1 pad 36: /RXB -> /A11
- J1 pad 37: /USR1 -> /A12
- J1 pad 38: /USR2 -> /A13
- J1 pad 39: /USR3 -> /A14
- J1 pad 4: /A12 -> /USR1
- J1 pad 40: /USR4 -> /A15
- J1 pad 5: /A11 -> /RXB
- J1 pad 6: /A10 -> /TXB
- J1 pad 7: /A9 -> /RD
- J1 pad 8: /A8 -> /IORQ
- J1 pad 9: /A7 -> /WR
- J3 pad 1: /A15 -> /USR4
- J3 pad 10: /A6 -> /MREQ
- J3 pad 11: /A5 -> /INT
- J3 pad 12: /A4 -> /RST
- J3 pad 13: /A3 -> /M1
- J3 pad 14: /A2 -> /CLK
- J3 pad 15: /A1 -> /D0
- J3 pad 16: /A0 -> /D1
- J3 pad 17: VCC -> /D2
- J3 pad 18: GND -> /D3
- J3 pad 19: /D7 -> /D4
- J3 pad 2: /A14 -> /USR3
- J3 pad 20: /D6 -> /D5
- J3 pad 21: /D5 -> /D6
- J3 pad 22: /D4 -> /D7
- J3 pad 23: /D3 -> GND
- J3 pad 24: /D2 -> VCC
- J3 pad 25: /D1 -> /A0
- J3 pad 26: /D0 -> /A1
- J3 pad 27: /CLK -> /A2
- J3 pad 28: /M1 -> /A3
- J3 pad 29: /RST -> /A4
- J3 pad 3: /A13 -> /USR2
- J3 pad 30: /INT -> /A5
- J3 pad 31: /MREQ -> /A6
- J3 pad 32: /WR -> /A7
- J3 pad 33: /IORQ -> /A8
- J3 pad 34: /RD -> /A9
- J3 pad 35: /TXB -> /A10
- J3 pad 36: /RXB -> /A11
- J3 pad 37: /USR1 -> /A12
- J3 pad 38: /USR2 -> /A13
- J3 pad 39: /USR3 -> /A14
- J3 pad 4: /A12 -> /USR1
- J3 pad 40: /USR4 -> /A15
- J3 pad 5: /A11 -> /RXB
- J3 pad 6: /A10 -> /TXB
- J3 pad 7: /A9 -> /RD
- J3 pad 8: /A8 -> /IORQ
- J3 pad 9: /A7 -> /WR
- J5 pad 1: /A15 -> /USR4
- J5 pad 10: /A6 -> /MREQ
- J5 pad 11: /A5 -> /INT
- J5 pad 12: /A4 -> /RST
- J5 pad 13: /A3 -> /M1
- J5 pad 14: /A2 -> /CLK
- J5 pad 15: /A1 -> /D0
- J5 pad 16: /A0 -> /D1
- J5 pad 17: VCC -> /D2
- J5 pad 18: GND -> /D3
- J5 pad 19: /D7 -> /D4
- J5 pad 2: /A14 -> /USR3
- J5 pad 20: /D6 -> /D5
- J5 pad 21: /D5 -> /D6
- J5 pad 22: /D4 -> /D7
- J5 pad 23: /D3 -> GND
- J5 pad 24: /D2 -> VCC
- J5 pad 25: /D1 -> /A0
- J5 pad 26: /D0 -> /A1
- J5 pad 27: /CLK -> /A2
- J5 pad 28: /M1 -> /A3
- J5 pad 29: /RST -> /A4
- J5 pad 3: /A13 -> /USR2
- J5 pad 30: /INT -> /A5
- J5 pad 31: /MREQ -> /A6
- J5 pad 32: /WR -> /A7
- J5 pad 33: /IORQ -> /A8
- J5 pad 34: /RD -> /A9
- J5 pad 35: /TXB -> /A10
- J5 pad 36: /RXB -> /A11
- J5 pad 37: /USR1 -> /A12
- J5 pad 38: /USR2 -> /A13
- J5 pad 39: /USR3 -> /A14
- J5 pad 4: /A12 -> /USR1
- J5 pad 40: /USR4 -> /A15
- J5 pad 5: /A11 -> /RXB
- J5 pad 6: /A10 -> /TXB
- J5 pad 7: /A9 -> /RD
- J5 pad 8: /A8 -> /IORQ
- J5 pad 9: /A7 -> /WR
- J7 pad 1: /A15 -> /USR4
- J7 pad 10: /A6 -> /MREQ
- J7 pad 11: /A5 -> /INT
- J7 pad 12: /A4 -> /RST
- J7 pad 13: /A3 -> /M1
- J7 pad 14: /A2 -> /CLK
- J7 pad 15: /A1 -> /D0
- J7 pad 16: /A0 -> /D1
- J7 pad 17: VCC -> /D2
- J7 pad 18: GND -> /D3
- J7 pad 19: /D7 -> /D4
- J7 pad 2: /A14 -> /USR3
- J7 pad 20: /D6 -> /D5
- J7 pad 21: /D5 -> /D6
- J7 pad 22: /D4 -> /D7
- J7 pad 23: /D3 -> GND
- J7 pad 24: /D2 -> VCC
- J7 pad 25: /D1 -> /A0
- J7 pad 26: /D0 -> /A1
- J7 pad 27: /CLK -> /A2
- J7 pad 28: /M1 -> /A3
- J7 pad 29: /RST -> /A4
- J7 pad 3: /A13 -> /USR2
- J7 pad 30: /INT -> /A5
- J7 pad 31: /MREQ -> /A6
- J7 pad 32: /WR -> /A7
- J7 pad 33: /IORQ -> /A8
- J7 pad 34: /RD -> /A9
- J7 pad 35: /TXB -> /A10
- J7 pad 36: /RXB -> /A11
- J7 pad 37: /USR1 -> /A12
- J7 pad 38: /USR2 -> /A13
- J7 pad 39: /USR3 -> /A14
- J7 pad 4: /A12 -> /USR1
- J7 pad 40: /USR4 -> /A15
- J7 pad 5: /A11 -> /RXB
- J7 pad 6: /A10 -> /TXB
- J7 pad 7: /A9 -> /RD
- J7 pad 8: /A8 -> /IORQ
- J7 pad 9: /A7 -> /WR
- J9 pad 1: /A15 -> /USR4
- J9 pad 10: /A6 -> /MREQ
- J9 pad 11: /A5 -> /INT
- J9 pad 12: /A4 -> /RST
- J9 pad 13: /A3 -> /M1
- J9 pad 14: /A2 -> /CLK
- J9 pad 15: /A1 -> /D0
- J9 pad 16: /A0 -> /D1
- J9 pad 17: VCC -> /D2
- J9 pad 18: GND -> /D3
- J9 pad 19: /D7 -> /D4
- J9 pad 2: /A14 -> /USR3
- J9 pad 20: /D6 -> /D5
- J9 pad 21: /D5 -> /D6
- J9 pad 22: /D4 -> /D7
- J9 pad 23: /D3 -> GND
- J9 pad 24: /D2 -> VCC
- J9 pad 25: /D1 -> /A0
- J9 pad 26: /D0 -> /A1
- J9 pad 27: /CLK -> /A2
- J9 pad 28: /M1 -> /A3
- J9 pad 29: /RST -> /A4
- J9 pad 3: /A13 -> /USR2
- J9 pad 30: /INT -> /A5
- J9 pad 31: /MREQ -> /A6
- J9 pad 32: /WR -> /A7
- J9 pad 33: /IORQ -> /A8
- J9 pad 34: /RD -> /A9
- J9 pad 35: /TXB -> /A10
- J9 pad 36: /RXB -> /A11
- J9 pad 37: /USR1 -> /A12
- J9 pad 38: /USR2 -> /A13
- J9 pad 39: /USR3 -> /A14
- J9 pad 4: /A12 -> /USR1
- J9 pad 40: /USR4 -> /A15
- J9 pad 5: /A11 -> /RXB
- J9 pad 6: /A10 -> /TXB
- J9 pad 7: /A9 -> /RD
- J9 pad 8: /A8 -> /IORQ
- J9 pad 9: /A7 -> /WR

Commit message: Added CERN license text to silkscreen
Other:
- board text added: "Licensed under CERN-OHL-S v2"
Changed lines of the file:
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@@
   (general
     (thickness 1.6)
-    (drawings 76)
+    (drawings 77)
     (tracks 743)
     (zones 0)
@@
     )
   )
+  (gr_text "Licensed under CERN-OHL-S v2" (at 107.315 139.7) (layer B.SilkS)
+    (effects (font (size 1 1) (thickness 0.15)) (justify mirror))
+  )
   (gr_text Switch (at 144.78 137.795) (layer F.SilkS)

Commit message: Finished Backplane
Parts:
- R3: moved to F.Cu
- moved R3 6.35 mm to (154.3, 134.0), turned to 270 degrees
Routing:
- net Net-(J12-Pad1): track 9.03 -> 3.28 mm
- net VCC: track 308.9 -> 312.0 mm

Commit message: Updated Backplane
Connections:
- J10 pad 1: Net-(J10-Pad1) -> VCC
- J2 pad 1: VCC -> Net-(J2-Pad1)
- J4 pad 1: Net-(J2-Pad2) -> Net-(J4-Pad1)
- J4 pad 2: Net-(J4-Pad2) -> Net-(J2-Pad1)
- J6 pad 1: Net-(J4-Pad2) -> Net-(J6-Pad1)
- J6 pad 2: Net-(J6-Pad2) -> Net-(J4-Pad1)
- J8 pad 1: Net-(J6-Pad2) -> Net-(J10-Pad2)
- J8 pad 2: Net-(J10-Pad1) -> Net-(J6-Pad1)
Routing:
- net VCC: track 312.0 -> 332.0 mm
- net Net-(J2-Pad2): track 16.3 -> 0.00 mm
- net Net-(J2-Pad1): track 0.00 -> 16.3 mm
- net Net-(J10-Pad2): track 0.00 -> 16.3 mm
- net Net-(J10-Pad1): track 16.3 -> 0.00 mm
- net Net-(J6-Pad2): track 16.3 -> 0.00 mm
- net Net-(J6-Pad1): track 0.00 -> 16.3 mm
- net Net-(J4-Pad1): track 0.00 -> 16.3 mm
- net Net-(J4-Pad2): track 16.3 -> 0.00 mm
